File: Arduino Shield.brd (EAGLE design)
At the start: 59.7 x 53.4 mm, 8 parts

Commit message: Update Arduino Shield.brd
Routing:
- removed copper zone on layer 1, net GND
Other:
- board size 59.7 x 53.4 mm -> 59.7 x 53.3 mm
Changed lines of the file:
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@@
 <board>
 <plain>
-<wire x1="0" y1="0" x2="59.67" y2="0" width="0" layer="20"/>
-<wire x1="59.67" y1="0" x2="59.67" y2="53.391" width="0" layer="20"/>
-<wire x1="59.67" y1="53.391" x2="0" y2="53.391" width="0" layer="20"/>
-<wire x1="0" y1="53.391" x2="0" y2="0" width="0" layer="20"/>
+<wire x1="0" y1="2.54" x2="0" y2="50.8" width="0.1524" layer="20"/>
+<wire x1="0" y1="50.8" x2="2.54" y2="53.34" width="0.1524" layer="20"/>
+<wire x1="2.54" y1="53.34" x2="55.88" y2="53.34" width="0.1524" layer="20"/>
+<wire x1="55.88" y1="53.34" x2="57.15" y2="52.07" width="0.1524" layer="20"/>
+<wire x1="57.15" y1="52.07" x2="57.15" y2="40.64" width="0.1524" layer="20"/>
+<wire x1="57.15" y1="40.64" x2="59.69" y2="38.1" width="0.1524" layer="20"/>
+<wire x1="59.69" y1="38.1" x2="59.69" y2="5.08" width="0.1524" layer="20"/>
+<wire x1="59.69" y1="5.08" x2="57.15" y2="2.54" width="0.1524" layer="20"/>
+<wire x1="57.15" y1="2.54" x2="57.15" y2="0" width="0.1524" layer="20"/>
+<wire x1="57.15" y1="0" x2="2.54" y2="0" width="0.1524" layer="20"/>
+<wire x1="2.54" y1="0" x2="0" y2="2.54" width="0.1524" layer="20"/>
 </plain>
 <attributes>
@@
 <vertex x="2.54" y="53.34"/>
 </polygon>
-<polygon width="0.508" layer="1" isolate="0.4064">
+<polygon width="0.508" layer="16" isolate="0.4064">
 <vertex x="0" y="50.8"/>
 <vertex x="0" y="2.54"/>
